Commit message: Updated arm functionality for mpo_700 and mpo_500; restructured pkg; modularized mpo_500 urdf to xacro

File: components/common_macro/gazebo_lidar_macro.xacro (robot description, xacro)
@@ -1,4 +1,4 @@
 <?xml version="1.0"?>
-<robot xmlns:xacro="http://www.ros.org/wiki/xacro" name="mpo_700">
+<robot xmlns:xacro="http://www.ros.org/wiki/xacro" name="mpo">
     <xacro:macro name="gazebo_lidar_sensor" params="
       sensor_name

File: components/common_macro/gazebo_object_controller_macro.xacro (robot description, xacro)
@@ -1,4 +1,4 @@
 <?xml version="1.0"?>
-<robot xmlns:xacro="http://www.ros.org/wiki/xacro" name="mpo_700">
+<robot xmlns:xacro="http://www.ros.org/wiki/xacro" name="mpo">
     <!--Gazebo Object Controller Macro-->
     <xacro:macro name="gazebo_object_controller" params="
@@ -7,4 +7,5 @@
         odom_frame
         base_frame
+        covariance_yaw
         ">
         <gazebo>
@@ -27,5 +28,5 @@
                 <covariance_x>0.0001</covariance_x>
                 <covariance_y>0.0001</covariance_y>
-                <covariance_yaw>0.0001</covariance_yaw>
+                <covariance_yaw>${covariance_yaw}</covariance_yaw>
             </plugin>
         </gazebo>

File: robots/mpo_500/mpo_500.urdf.xacro (robot description, xacro)
@@ -1,5 +1,5 @@
 <?xml version="1.0"?>
-<!-- This is the main URDF file for mpo_700-->
-<robot xmlns:xacro="http://www.ros.org/wiki/xacro" name="mpo_700">
+<!-- This is the main URDF file for mpo_500-->
+<robot xmlns:xacro="http://www.ros.org/wiki/xacro" name="mpo_500">
     <!--set use_gazebo = false for implementation on real robot-->
     <xacro:arg name="use_gazebo" default="true"/>
@@ -9,10 +9,7 @@
     <xacro:property name="model_scale" value="0.001 0.001 0.001" />
     <!-- Base Properties -->
-    <xacro:property name= "base_link_mass" value="140" />
+    <xacro:property name= "base_link_mass" value="64" />
     <!-- Wheel Properties -->
-    <xacro:property name="wheel_link_mass" value="1.2" />
-    <!-- caster Wheel Properties -->
-    <xacro:property name="caster_inertial_value" value="0.27258101" />
-    <xacro:property name="caster_link_mass" value="12.7" />
+    <xacro:property name="wheel_link_mass" value="2.2" />
     <!-- Arm properties-->
     <xacro:property name="arm" value="$(arg arm_type)"/>
@@ -29,8 +26,8 @@
     </xacro:unless>
     <!-- import main body description -->
-    <xacro:include filename="$(find neo_simulation2)/robots/mpo_700/urdf/mpo_700_body.urdf.xacro"/>
+    <xacro:include filename="$(find neo_simulation2)/robots/mpo_500/urdf/mpo_500_body.urdf.xacro"/>
     <!-- If Simulation is used -->
     <xacro:if value="$(arg use_gazebo)">
-        <xacro:include filename="$(find neo_simulation2)/robots/mpo_700/urdf/mpo_700_gazebo.urdf.xacro"/>
+        <xacro:include filename="$(find neo_simulation2)/robots/mpo_500/urdf/mpo_500_gazebo.urdf.xacro"/>
     </xacro:if>
     <!-- Check if one of the arms is used -->
@@ -43,12 +40,12 @@
         <xacro:include filename="$(find neo_simulation2)/components/common_macro/mpo_cabinet_macro.xacro"/>
         <xacro:cabinet
-            neo_robot_name="mpo_700"
+            neo_robot_name="mpo_500"
             parent_link="base_link"
             model_scale="${model_scale}"
-            inertial_rpy="0 0 -1.5708"
+            inertial_rpy="0 0 0"
             visual_rpy="0 0 -1.5708"
-            collision_rpy="0 0 -1.5708"
+            collision_rpy="0 0 0"
         >
-            <origin rpy="0 0 0" xyz="0.025 0 0.35"/>
+            <origin rpy="0 0 0" xyz="0.072 0 0.386"/>
         </xacro:cabinet>
         <!-- Universal Robotics Arm-->
@@ -61,6 +58,3 @@
         </xacro:if>
     </xacro:if>
-      <!-- SENSORS -->
-      <!-- Sick S300 - Comment/Uncomment if required -->
-      <!-- <xacro:include filename="$(find neo_simulation2)/robots/mpo_700/xacros/sick_S300.xacro" /> -->
 </robot>

File: robots/mpo_500/urdf/macro/mpo_500_wheel_macro.xacro (robot description, xacro)
@@ -2,13 +2,9 @@
 <robot xmlns:xacro="http://www.ros.org/wiki/xacro" name="mpo_700">
     <!--WHEEL MACRO-->
-    <xacro:macro name="mpo_700_wheel" params="
+    <xacro:macro name="mpo_500_wheel" params="
         wheel_prefix
-        parent_prefix
-        link_origin_rpy
+        parent_link
         *origin
         wheel_joint_type
-        ixx
-        iyy
-        izz
         has_limits
         model_scale
@@ -19,17 +15,16 @@
                 <mass value="${wheel_link_mass}"/>
                 <origin rpy="0 0 0" xyz="0 0 0"/>
-                <inertia ixx="${ixx}" ixy="0" ixz="0" iyy="${iyy}" iyz="0" izz="${izz}"/>
+                <inertia ixx="0.01" ixy="0.0" ixz="0.0" iyy="0.01" iyz="0.0" izz="0.01"/>
             </inertial>
             <visual>
-                <origin rpy="${link_origin_rpy}" xyz="0 0 0"/>
+                <origin rpy="0 0 0" xyz="0 0 0"/>
                 <geometry>
-                    <mesh filename="package://neo_simulation2/robots/mpo_700/meshes/MPO-700-WHEEL.dae" scale="${model_scale}"/>
+                    <mesh filename="package://neo_simulation2/robots/mpo_500/meshes/MPO-500-WHEEL.dae" scale="${model_scale}"/>
                 </geometry>
             </visual>
             <collision>
-                <origin rpy="0 0 0" xyz="0 0 0"/>
+                <origin rpy="0 1.57 1.57" xyz="0 0 0"/>
                 <geometry>
-                    <sphere radius="0.09"/>
-                    <!-- <mesh filename="package://neo_simulation2/robots/mpo_700/meshes/MPO-700-WHEEL.dae" scale="${model_scale}"/> -->
+                    <sphere radius="0.117"/>
                 </geometry>
             </collision>
@@ -39,9 +34,9 @@
             <xacro:insert_block name="origin"/>
             <xacro:if value="${has_limits}">
-                <limit effort="1000.0" lower="-1e+16" upper="1e+16" velocity="20.5"/>
+                <limit effort="1000.0" lower="-1e+16" upper="1e+16" velocity="15"/>
             </xacro:if>
-            <axis xyz="0 -1 0"/>
-            <joint_properties damping="30" friction="110"/>
-            <parent link="${parent_prefix}_link"/>
+            <axis xyz="0 1 0"/>
+            <joint_properties damping="1.0" friction="1"/>
+            <parent link="${parent_link}"/>
             <child link="${wheel_prefix}_link"/>
         </joint>

File: robots/mpo_500/urdf/mpo_500_gazebo.urdf.xacro (robot description, xacro)
@@ -1,12 +1,12 @@
 <?xml version="1.0"?>
-<robot xmlns:xacro="http://www.ros.org/wiki/xacro" name="mpo_700">
+<robot xmlns:xacro="http://www.ros.org/wiki/xacro" name="mpo_500">
     <!-- Include macros -->
     <xacro:include filename="$(find neo_simulation2)/components/common_macro/gazebo_lidar_macro.xacro" />
     <xacro:include filename="$(find neo_simulation2)/components/common_macro/gazebo_object_controller_macro.xacro" />
-    <xacro:include filename="$(find neo_simulation2)/robots/mpo_700/urdf/macro/gazebo_mpo_700_wheel_macro.xacro" />
+    <xacro:include filename="$(find neo_simulation2)/robots/mpo_500/urdf/macro/gazebo_mpo_500_wheel_macro.xacro" />
     <!-- Properties -->
     <xacro:property name="wheel_mu" value="0.0001" />
-    <xacro:property name="lidar_1_update_rate" value="40" />
-    <xacro:property name="lidar_2_update_rate" value="40" />
+    <xacro:property name="lidar_1_update_rate" value="100" />
+    <xacro:property name="lidar_2_update_rate" value="100" />
     <xacro:property name="controller_update_rate" value="100" />
     <xacro:property name="odom_update_rate" value="100" />
@@ -16,6 +16,6 @@
         controller_update_rate="${controller_update_rate}"
         odom_frame="odom"
-        base_frame="base_footprint"
-        covariance_yaw="0.0001"
+        base_frame="base_link"
+        covariance_yaw="0.01"
     />
     <!--Lidar Sensors-->
@@ -32,5 +32,5 @@
         noise_stddev="0.01"
         topic_name="scan"
-        visualize="false"
+        visualize="true"
     />
     <xacro:gazebo_lidar_sensor
@@ -46,26 +46,22 @@
         noise_stddev="0.01"
         topic_name="scan2"
-        visualize="false"
+        visualize="true"
     />
     <!--Wheels-->
-    <xacro:gazebo_mpo_700_wheel
-        wheel_prefix="mpo_700_wheel_front_right"
+    <xacro:gazebo_mpo_500_wheel
+        wheel_prefix="mpo_500_omni_wheel_front_right"
         wheel_mu="${wheel_mu}"
         />
-    <xacro:gazebo_mpo_700_wheel
-        wheel_prefix="mpo_700_wheel_back_right"
+    <xacro:gazebo_mpo_500_wheel
+        wheel_prefix="mpo_500_omni_wheel_back_right"
         wheel_mu="${wheel_mu}"
         />
-    <xacro:gazebo_mpo_700_wheel
-        wheel_prefix="mpo_700_wheel_front_left"
+    <xacro:gazebo_mpo_500_wheel
+        wheel_prefix="mpo_500_omni_wheel_front_left"
         wheel_mu="${wheel_mu}"
         />
-    <xacro:gazebo_mpo_700_wheel
-        wheel_prefix="mpo_700_wheel_back_left"
+    <xacro:gazebo_mpo_500_wheel
+        wheel_prefix="mpo_500_omni_wheel_back_left"
         wheel_mu="${wheel_mu}"
         />
-    <!-- SENSORS -->
-    <!-- Sick S300 - Comment/Uncomment if required -->
-    <!-- <xacro:include filename="$(find neo_simulation2)/robots/mpo_700/xacros/sick_S300.xacro" /> -->
-    <!--Ultrasonics, cameras and IMU's  -->
 </robot>

File: robots/mpo_700/urdf/mpo_700_body.urdf.xacro (robot description, xacro)
@@ -45,5 +45,5 @@
             <origin rpy="-1.57 0 3.14" xyz="0 0 -0.12"/>
             <geometry>
-                <mesh filename="package://neo_simulation2/components/sensors/SICK-S300.dae" scale="${model_scale}"/>
+                <mesh filename="package://neo_simulation2/components/meshes/SICK-S300.dae" scale="${model_scale}"/>
             </geometry>
         </visual>
@@ -51,5 +51,5 @@
             <origin rpy="-1.57 0 3.14" xyz="0 0 -0.12"/>
             <geometry>
-                <mesh filename="package://neo_simulation2/components/sensors/SICK-S300.dae" scale="${model_scale}"/>
+                <mesh filename="package://neo_simulation2/components/meshes/SICK-S300.dae" scale="${model_scale}"/>
             </geometry>
         </collision>
@@ -70,5 +70,5 @@
             <origin rpy="-1.57 0 3.14" xyz="0 0 -0.12"/>
             <geometry>
-                <mesh filename="package://neo_simulation2/components/sensors/SICK-S300.dae" scale="${model_scale}"/>
+                <mesh filename="package://neo_simulation2/components/meshes/SICK-S300.dae" scale="${model_scale}"/>
             </geometry>
         </visual>
@@ -76,5 +76,5 @@
             <origin rpy="-1.57 0 3.14" xyz="0 0 -0.12"/>
             <geometry>
-                <mesh filename="package://neo_simulation2/components/sensors/SICK-S300.dae" scale="${model_scale}"/>
+                <mesh filename="package://neo_simulation2/components/meshes/SICK-S300.dae" scale="${model_scale}"/>
             </geometry>
         </collision>
@@ -85,5 +85,5 @@
     <!-- Caster wheels -->
     <xacro:mpo_700_caster_wheel
-        caster_prefix="caster_front_left"
+        caster_prefix="mpo_700_caster_front_left"
         caster_joint_type="${ODM_joint_type}"
         link_origin_rpy="0 0 0"
@@ -97,5 +97,5 @@
     </xacro:mpo_700_caster_wheel>
     <xacro:mpo_700_caster_wheel
-        caster_prefix="caster_front_right"
+        caster_prefix="mpo_700_caster_front_right"
         caster_joint_type="${ODM_joint_type}"
         link_origin_rpy="0 0 3.14"
@@ -109,5 +109,5 @@
     </xacro:mpo_700_caster_wheel>
     <xacro:mpo_700_caster_wheel
-        caster_prefix="caster_back_left"
+        caster_prefix="mpo_700_caster_back_left"
         caster_joint_type="${ODM_joint_type}"
         link_origin_rpy="0 0 0"
@@ -121,5 +121,5 @@
     </xacro:mpo_700_caster_wheel>
     <xacro:mpo_700_caster_wheel
-        caster_prefix="caster_back_right"
+        caster_prefix="mpo_700_caster_back_right"
         caster_joint_type="${ODM_joint_type}"
         link_origin_rpy="0 0 3.14"
@@ -134,6 +134,6 @@
     <!-- NOTE: All wheels have limits-->
     <xacro:mpo_700_wheel
-        wheel_prefix="wheel_front_left"
-        parent_link="caster_front_left"
+        wheel_prefix="mpo_700_wheel_front_left"
+        parent_prefix="mpo_700_caster_front_left"
         wheel_joint_type="${ODM_joint_type}"
         link_origin_rpy="0 0 3.14"
@@ -147,6 +147,6 @@
     </xacro:mpo_700_wheel>
     <xacro:mpo_700_wheel
-        wheel_prefix="wheel_front_right"
-        parent_link="caster_front_right"
+        wheel_prefix="mpo_700_wheel_front_right"
+        parent_prefix="mpo_700_caster_front_right"
         wheel_joint_type="${ODM_joint_type}"
         link_origin_rpy="0 0 3.14"
@@ -160,6 +160,6 @@
     </xacro:mpo_700_wheel>
     <xacro:mpo_700_wheel
-        wheel_prefix="wheel_back_left"
-        parent_link="caster_back_left"
+        wheel_prefix="mpo_700_wheel_back_left"
+        parent_prefix="mpo_700_caster_back_left"
         wheel_joint_type="${ODM_joint_type}"
         link_origin_rpy="0 0 3.14"
@@ -173,6 +173,6 @@
     </xacro:mpo_700_wheel>
     <xacro:mpo_700_wheel
-        wheel_prefix="wheel_back_right"
-        parent_link="caster_back_right"
+        wheel_prefix="mpo_700_wheel_back_right"
+        parent_prefix="mpo_700_caster_back_right"
         wheel_joint_type="${ODM_joint_type}"
         link_origin_rpy="0 0 3.14"
