Commit message: modified mpo_700 and mpo_500 urdf and parameters

File: components/common_macro/mpo_cabinet_macro.xacro (robot description, xacro)
@@ -19,5 +19,5 @@
         <link name="cabinet_link">
             <inertial>
-                <mass value="2"/>
+                <mass value="10"/>
                 <origin rpy="${inertial_rpy}" xyz="0 0 0"/>
                 <inertia ixx="0.457072" ixy="0.0" ixz="0.0" iyy="0.23616" iyz="0.0" izz="0.686"/>

File: robots/mpo_500/mpo_500.urdf.xacro (robot description, xacro)
@@ -6,10 +6,4 @@
     <!--set arm name to include the arm in the simulation-->
     <xacro:arg name="arm_type" default=""/>
-    <!-- Model Scale -->
-    <xacro:property name="model_scale" value="0.001 0.001 0.001" />
-    <!-- Base Properties -->
-    <xacro:property name= "base_link_mass" value="64" />
-    <!-- Wheel Properties -->
-    <xacro:property name="wheel_link_mass" value="2.2" />
     <!-- Arm properties-->
     <xacro:property name="arm" value="$(arg arm_type)"/>
@@ -42,5 +36,5 @@
             neo_robot_name="mpo_500"
             parent_link="base_link"
-            model_scale="${model_scale}"
+            model_scale="0.001 0.001 0.001"
             inertial_rpy="0 0 0"
             visual_rpy="0 0 -1.5708"

File: robots/mpo_500/urdf/macro/gazebo_mpo_500_wheel_macro.xacro (robot description, xacro)
@@ -4,5 +4,4 @@
     <xacro:macro name="gazebo_mpo_500_wheel" params="
       wheel_prefix
-      wheel_mu
       ">
         <gazebo reference="${wheel_prefix}_link">
@@ -10,6 +9,8 @@
             <!-- <fdir1>0 1 0</fdir1> -->
             <!-- <slip1> 0.1 </slip1> -->
-            <mu1>${wheel_mu}</mu1>
-            <mu2>${wheel_mu}</mu2>
+            <mu1>0.045</mu1>
+            <mu2>0.045</mu2>
+            <kp>100000.0</kp>
+            <kd>10.0</kd>
         </gazebo>
     </xacro:macro>

File: robots/mpo_500/urdf/macro/mpo_500_wheel_macro.xacro (robot description, xacro)
@@ -2,5 +2,5 @@
 <robot xmlns:xacro="http://www.ros.org/wiki/xacro" name="mpo_700">
     <!--WHEEL MACRO-->
-    <xacro:macro name="mpo_500_wheel" params="
+    <xacro:macro name="mpo_500_omni_wheel" params="
         wheel_prefix
         parent_link
@@ -13,5 +13,5 @@
         <link name="${wheel_prefix}_link" type="wheel">
             <inertial>
-                <mass value="${wheel_link_mass}"/>
+                <mass value="2.2"/>
                 <origin rpy="0 0 0" xyz="0 0 0"/>
                 <inertia ixx="0.01" ixy="0.0" ixz="0.0" iyy="0.01" iyz="0.0" izz="0.01"/>

File: robots/mpo_500/urdf/mpo_500_body.urdf.xacro (robot description, xacro)
@@ -12,5 +12,5 @@
     <link name="base_link">
         <inertial>
-            <mass value="${base_link_mass}"/>
+            <mass value="64"/>
             <origin xyz="0 0 0"/>
             <inertia ixx="2.8" ixy="0.0" ixz="0.0" iyy="2.8" iyz="0.0" izz="2.8"/>
@@ -19,5 +19,5 @@
             <origin rpy="-1.571 0 1.571" xyz="0. 0. 0"/>
             <geometry>
-                <mesh filename="package://neo_simulation2/robots/mpo_500/meshes/MPO-500-BODY.dae" scale="${model_scale}"/>
+                <mesh filename="package://neo_simulation2/robots/mpo_500/meshes/MPO-500-BODY.dae" scale="0.001 0.001 0.001"/>
             </geometry>
         </visual>
@@ -25,5 +25,5 @@
             <origin rpy="-1.571 0 1.571" xyz="0. 0. 0"/>
             <geometry>
-                <mesh filename="package://neo_simulation2/robots/mpo_500/meshes/MPO-500-BODY.dae" scale="${model_scale}"/>
+                <mesh filename="package://neo_simulation2/robots/mpo_500/meshes/MPO-500-BODY.dae" scale="0.001 0.001 0.001"/>
             </geometry>
         </collision>
@@ -45,5 +45,5 @@
             <origin rpy="1.57 0 0" xyz="0 0 -0.06"/>
             <geometry>
-                <mesh filename="package://neo_simulation2/components/meshes/SICK-MICROSCAN3.dae" scale="${model_scale}"/>
+                <mesh filename="package://neo_simulation2/components/meshes/SICK-MICROSCAN3.dae" scale="0.001 0.001 0.001"/>
             </geometry>
         </visual>
@@ -51,5 +51,5 @@
             <origin rpy="1.57 0 0" xyz="0 0 -0.06"/>
             <geometry>
-                <mesh filename="package://neo_simulation2/components/meshes/SICK-MICROSCAN3.dae" scale="${model_scale}"/>
+                <mesh filename="package://neo_simulation2/components/meshes/SICK-MICROSCAN3.dae" scale="0.001 0.001 0.001"/>
             </geometry>
         </collision>
@@ -70,5 +70,5 @@
             <origin rpy="1.57 0 0" xyz="0 0 -0.06"/>
             <geometry>
-                <mesh filename="package://neo_simulation2/components/meshes/SICK-MICROSCAN3.dae" scale="${model_scale}"/>
+                <mesh filename="package://neo_simulation2/components/meshes/SICK-MICROSCAN3.dae" scale="0.001 0.001 0.001"/>
             </geometry>
         </visual>
@@ -76,5 +76,5 @@
             <origin rpy="1.57 0 0" xyz="0 0 -0.06"/>
             <geometry>
-                <mesh filename="package://neo_simulation2/components/meshes/SICK-MICROSCAN3.dae" scale="${model_scale}"/>
+                <mesh filename="package://neo_simulation2/components/meshes/SICK-MICROSCAN3.dae" scale="0.001 0.001 0.001"/>
             </geometry>
         </collision>
@@ -83,39 +83,39 @@
     <xacro:include filename="$(find neo_simulation2)/robots/mpo_500/urdf/macro/mpo_500_wheel_macro.xacro"/>
     <!-- Omni Wheels-->
-    <xacro:mpo_500_wheel
+    <xacro:mpo_500_omni_wheel
         wheel_prefix="mpo_500_omni_wheel_front_left"
         parent_link="base_link"
         wheel_joint_type="${ODM_joint_type}"
         has_limits="true"
-        model_scale="${model_scale}"
+        model_scale="0.001 0.001 0.001"
         >
         <origin rpy="0 0 0" xyz="0.25 0.28 0.13"/>
-    </xacro:mpo_500_wheel>
-    <xacro:mpo_500_wheel
+    </xacro:mpo_500_omni_wheel>
+    <xacro:mpo_500_omni_wheel
         wheel_prefix="mpo_500_omni_wheel_front_right"
         parent_link="base_link"
         wheel_joint_type="${ODM_joint_type}"
         has_limits="true"
-        model_scale="${model_scale}"
+        model_scale="0.001 0.001 0.001"
         >
         <origin rpy="0 0 3.14" xyz="0.25 -0.28 0.13"/>
-    </xacro:mpo_500_wheel>
-    <xacro:mpo_500_wheel
+    </xacro:mpo_500_omni_wheel>
+    <xacro:mpo_500_omni_wheel
         wheel_prefix="mpo_500_omni_wheel_back_left"
         parent_link="base_link"
         wheel_joint_type="${ODM_joint_type}"
         has_limits="true"
-        model_scale="${model_scale}"
+        model_scale="0.001 0.001 0.001"
         >
         <origin rpy="0 0 0" xyz="-0.25 0.28 0.13"/>
-    </xacro:mpo_500_wheel>
-    <xacro:mpo_500_wheel
+    </xacro:mpo_500_omni_wheel>
+    <xacro:mpo_500_omni_wheel
         wheel_prefix="mpo_500_omni_wheel_back_right"
         parent_link="base_link"
         wheel_joint_type="${ODM_joint_type}"
         has_limits="true"
-        model_scale="${model_scale}"
+        model_scale="0.001 0.001 0.001"
         >
         <origin rpy="0 0 3.14" xyz="-0.25 -0.28 0.13"/>
-    </xacro:mpo_500_wheel>
+    </xacro:mpo_500_omni_wheel>
 </robot>

File: robots/mpo_500/urdf/mpo_500_gazebo.urdf.xacro (robot description, xacro)
@@ -6,5 +6,4 @@
     <xacro:include filename="$(find neo_simulation2)/robots/mpo_500/urdf/macro/gazebo_mpo_500_wheel_macro.xacro" />
     <!-- Properties -->
-    <xacro:property name="wheel_mu" value="0.0001" />
     <xacro:property name="lidar_1_update_rate" value="100" />
     <xacro:property name="lidar_2_update_rate" value="100" />
@@ -51,17 +50,13 @@
     <xacro:gazebo_mpo_500_wheel
         wheel_prefix="mpo_500_omni_wheel_front_right"
-        wheel_mu="${wheel_mu}"
         />
     <xacro:gazebo_mpo_500_wheel
         wheel_prefix="mpo_500_omni_wheel_back_right"
-        wheel_mu="${wheel_mu}"
         />
     <xacro:gazebo_mpo_500_wheel
         wheel_prefix="mpo_500_omni_wheel_front_left"
-        wheel_mu="${wheel_mu}"
         />
     <xacro:gazebo_mpo_500_wheel
         wheel_prefix="mpo_500_omni_wheel_back_left"
-        wheel_mu="${wheel_mu}"
         />
 </robot>

File: robots/mpo_700/mpo_700.urdf.xacro (robot description, xacro)
@@ -6,13 +6,4 @@
     <!--set arm name to include the arm in the simulation-->
     <xacro:arg name="arm_type" default=""/>
-    <!-- Model Scale -->
-    <xacro:property name="model_scale" value="0.001 0.001 0.001" />
-    <!-- Base Properties -->
-    <xacro:property name= "base_link_mass" value="140" />
-    <!-- Wheel Properties -->
-    <xacro:property name="wheel_link_mass" value="1.2" />
-    <!-- caster Wheel Properties -->
-    <xacro:property name="caster_inertial_value" value="0.27258101" />
-    <xacro:property name="caster_link_mass" value="12.7" />
     <!-- Arm properties-->
     <xacro:property name="arm" value="$(arg arm_type)"/>
@@ -45,5 +36,5 @@
             neo_robot_name="mpo_700"
             parent_link="base_link"
-            model_scale="${model_scale}"
+            model_scale="0.001 0.001 0.001"
             inertial_rpy="0 0 -1.5708"
             visual_rpy="0 0 -1.5708"

File: robots/mpo_700/urdf/macro/gazebo_mpo_700_wheel_macro.xacro (robot description, xacro)
@@ -4,12 +4,10 @@
     <xacro:macro name="gazebo_mpo_700_wheel" params="
       wheel_prefix
-      wheel_mu
       ">
         <gazebo reference="${wheel_prefix}_link">
-            <!-- <kp> 10000 </kp> -->
-            <!-- <fdir1>0 1 0</fdir1> -->
-            <!-- <slip1> 0.1 </slip1> -->
-            <mu1>${wheel_mu}</mu1>
-            <mu2>${wheel_mu}</mu2>
+            <mu1>0.05</mu1>
+            <mu2>0.05</mu2>
+            <kp>100000.0</kp>
+            <kd>10.0</kd>
         </gazebo>
     </xacro:macro>

File: robots/mpo_700/urdf/macro/mpo_700_caster_wheel_macro.xacro (robot description, xacro)
@@ -9,5 +9,4 @@
         parent_link
         caster_inertial_value
-        caster_link_mass
         has_limits
         model_scale
@@ -15,5 +14,5 @@
         <link name="${caster_prefix}_link">
             <inertial>
-                <mass value="${caster_link_mass}"/>
+                <mass value="12.7"/>
                 <origin xyz="0 0 0" rpy="0 0 0"/>
                 <inertia ixx="${caster_inertial_value}" ixy="0" ixz="0" iyy="${caster_inertial_value}" iyz="0" izz="${caster_inertial_value}"/>

File: robots/mpo_700/urdf/macro/mpo_700_wheel_macro.xacro (robot description, xacro)
@@ -8,7 +8,4 @@
         *origin
         wheel_joint_type
-        ixx
-        iyy
-        izz
         has_limits
         model_scale
@@ -17,7 +14,7 @@
         <link name="${wheel_prefix}_link" type="wheel">
             <inertial>
-                <mass value="${wheel_link_mass}"/>
+                <mass value="1.2"/>
                 <origin rpy="0 0 0" xyz="0 0 0"/>
-                <inertia ixx="${ixx}" ixy="0" ixz="0" iyy="${iyy}" iyz="0" izz="${izz}"/>
+                <inertia ixx="0.11042056" ixy="0" ixz="0" iyy="0.11042056" iyz="0" izz="0.11042056"/>
             </inertial>
             <visual>

File: robots/mpo_700/urdf/mpo_700_body.urdf.xacro (robot description, xacro)
@@ -12,5 +12,5 @@
     <link name="base_link">
         <inertial>
-            <mass value="${base_link_mass}"/>
+            <mass value="140"/>
             <origin xyz="0 0 0"/>
             <inertia ixx="7.8" ixy="0.0" ixz="0" iyy="7.8" iyz="0.0" izz="7.8"/>
@@ -19,5 +19,5 @@
             <origin rpy="0 0 -1.571" xyz="0.0 0.0 0.0"/>
             <geometry>
-                <mesh filename="package://neo_simulation2/robots/mpo_700/meshes/MPO-700-BODY.dae" scale="${model_scale}"/>
+                <mesh filename="package://neo_simulation2/robots/mpo_700/meshes/MPO-700-BODY.dae" scale="0.001 0.001 0.001"/>
             </geometry>
         </visual>
@@ -25,5 +25,5 @@
             <origin rpy="0 0 -1.571" xyz="0. 0. 0."/>
             <geometry>
-                <mesh filename="package://neo_simulation2/robots/mpo_700/meshes/MPO-700-BODY.dae" scale="${model_scale}"/>
+                <mesh filename="package://neo_simulation2/robots/mpo_700/meshes/MPO-700-BODY.dae" scale="0.001 0.001 0.001"/>
             </geometry>
         </collision>
@@ -45,5 +45,5 @@
             <origin rpy="-1.57 0 3.14" xyz="0 0 -0.12"/>
             <geometry>
-                <mesh filename="package://neo_simulation2/components/meshes/SICK-S300.dae" scale="${model_scale}"/>
+                <mesh filename="package://neo_simulation2/components/meshes/SICK-S300.dae" scale="0.001 0.001 0.001"/>
             </geometry>
         </visual>
@@ -51,5 +51,5 @@
             <origin rpy="-1.57 0 3.14" xyz="0 0 -0.12"/>
             <geometry>
-                <mesh filename="package://neo_simulation2/components/meshes/SICK-S300.dae" scale="${model_scale}"/>
+                <mesh filename="package://neo_simulation2/components/meshes/SICK-S300.dae" scale="0.001 0.001 0.001"/>
             </geometry>
         </collision>
@@ -70,5 +70,5 @@
             <origin rpy="-1.57 0 3.14" xyz="0 0 -0.12"/>
             <geometry>
-                <mesh filename="package://neo_simulation2/components/meshes/SICK-S300.dae" scale="${model_scale}"/>
+                <mesh filename="package://neo_simulation2/components/meshes/SICK-S300.dae" scale="0.001 0.001 0.001"/>
             </geometry>
         </visual>
@@ -76,5 +76,5 @@
             <origin rpy="-1.57 0 3.14" xyz="0 0 -0.12"/>
             <geometry>
-                <mesh filename="package://neo_simulation2/components/meshes/SICK-S300.dae" scale="${model_scale}"/>
+                <mesh filename="package://neo_simulation2/components/meshes/SICK-S300.dae" scale="0.001 0.001 0.001"/>
             </geometry>
         </collision>
@@ -89,8 +89,7 @@
         link_origin_rpy="0 0 0"
         parent_link="base_link"
-        caster_inertial_value="${caster_inertial_value}"
-        caster_link_mass="${caster_link_mass}"
+        caster_inertial_value="0.27258101"
         has_limits="true"
-        model_scale="${model_scale}"
+        model_scale="0.001 0.001 0.001"
         >
         <origin rpy="0 0 0" xyz="0.24 0.18 0.22"/>
@@ -101,8 +100,7 @@
         link_origin_rpy="0 0 3.14"
         parent_link="base_link"
-        caster_inertial_value="${caster_inertial_value}"
-        caster_link_mass="${caster_link_mass}"
+        caster_inertial_value="0.27258101"
         has_limits="true"
-        model_scale="${model_scale}"
+        model_scale="0.001 0.001 0.001"
         >
         <origin rpy="0 0 0" xyz="0.24 -0.18 0.22"/>
@@ -113,8 +111,7 @@
         link_origin_rpy="0 0 0"
         parent_link="base_link"
-        caster_inertial_value="${caster_inertial_value}"
-        caster_link_mass="${caster_link_mass}"
+        caster_inertial_value="0.27258101"
         has_limits="true"
-        model_scale="${model_scale}"
+        model_scale="0.001 0.001 0.001"
         >
         <origin rpy="0 0 0" xyz="-0.24 0.18 0.22"/>
@@ -125,8 +122,7 @@
         link_origin_rpy="0 0 3.14"
         parent_link="base_link"
-        caster_inertial_value="${caster_inertial_value}"
-        caster_link_mass="${caster_link_mass}"
+        caster_inertial_value="0.27258101"
         has_limits="true"
-        model_scale="${model_scale}"
+        model_scale="0.001 0.001 0.001"
         >
         <origin rpy="0 0 0" xyz="-0.24 -0.18 0.22"/>
@@ -138,9 +134,6 @@
         wheel_joint_type="${ODM_joint_type}"
         link_origin_rpy="0 0 3.14"
-        ixx="0.11042056"
-        iyy="0.11042056"
-        izz="0.11042056"
         has_limits="true"
-        model_scale="${model_scale}"
+        model_scale="0.001 0.001 0.001"
         >
         <origin rpy="0 0 0" xyz="0.0 0.045 -0.12"/>
@@ -151,9 +144,6 @@
         wheel_joint_type="${ODM_joint_type}"
         link_origin_rpy="0 0 3.14"
-        ixx="0.11042056"
-        iyy="0.11042056"
-        izz="0.11042056"
         has_limits="true"
-        model_scale="${model_scale}"
+        model_scale="0.001 0.001 0.001"
         >
         <origin rpy="0 0 3.14" xyz="0.0 -0.045 -0.12"/>
@@ -164,9 +154,6 @@
         wheel_joint_type="${ODM_joint_type}"
         link_origin_rpy="0 0 3.14"
-        ixx="0.11042056"
-        iyy="0.11042056"
-        izz="0.11042056"
         has_limits="true"
-        model_scale="${model_scale}"
+        model_scale="0.001 0.001 0.001"
         >
         <origin rpy="0 0 0" xyz="0.0 0.045 -0.12"/>
@@ -177,9 +164,6 @@
         wheel_joint_type="${ODM_joint_type}"
         link_origin_rpy="0 0 3.14"
-        ixx="0.11042056"
-        iyy="0.11042056"
-        izz="0.11042056"
         has_limits="true"
-        model_scale="${model_scale}"
+        model_scale="0.001 0.001 0.001"
         >
         <origin rpy="0 0 3.14" xyz="0.0 -0.045 -0.12"/>

File: robots/mpo_700/urdf/mpo_700_gazebo.urdf.xacro (robot description, xacro)
@@ -6,5 +6,4 @@
     <xacro:include filename="$(find neo_simulation2)/robots/mpo_700/urdf/macro/gazebo_mpo_700_wheel_macro.xacro" />
     <!-- Properties -->
-    <xacro:property name="wheel_mu" value="0.0001" />
     <xacro:property name="lidar_1_update_rate" value="40" />
     <xacro:property name="lidar_2_update_rate" value="40" />
@@ -51,17 +50,13 @@
     <xacro:gazebo_mpo_700_wheel
         wheel_prefix="mpo_700_wheel_front_right"
-        wheel_mu="${wheel_mu}"
         />
     <xacro:gazebo_mpo_700_wheel
         wheel_prefix="mpo_700_wheel_back_right"
-        wheel_mu="${wheel_mu}"
         />
     <xacro:gazebo_mpo_700_wheel
         wheel_prefix="mpo_700_wheel_front_left"
-        wheel_mu="${wheel_mu}"
         />
     <xacro:gazebo_mpo_700_wheel
         wheel_prefix="mpo_700_wheel_back_left"
-        wheel_mu="${wheel_mu}"
         />
     <!-- SENSORS -->
