Commit message: Switched base_link and base_footprint to follow Nav2 convention

File: components/common_macro/gazebo_object_controller_macro.xacro (robot description, xacro)
@@ -24,5 +24,5 @@
                 <!-- Frame IDs -->
                 <odometryFrame>${odom_frame}</odometryFrame>
-                <robotBaseFrame>${base_frame}</robotBaseFrame>
+                <robot_base_frame>${base_frame}</robot_base_frame>
                 <!-- Set odom covariance -->
                 <covariance_x>0.0001</covariance_x>

File: robots/mpo_500/urdf/mpo_500_body.urdf.xacro (robot description, xacro)
@@ -2,12 +2,4 @@
 <robot xmlns:xacro="http://www.ros.org/wiki/xacro" name="mpo_500">
     <link name="base_footprint"/>
-    <joint name="base_footprint_joint" type="fixed">
-        <origin rpy="0 0 0" xyz="0 0 0"/>
-        <axis xyz="0 0 -1"/>
-        <!-- <limit effort="1000.0" lower="-1e+16" upper="1e+16" velocity="15"/> -->
-        <joint_properties damping="1" friction="1"/>
-        <parent link="base_footprint"/>
-        <child link="base_link"/>
-    </joint>
     <link name="base_link">
         <inertial>
@@ -29,4 +21,12 @@
         </collision>
     </link>
+    <joint name="base_footprint_joint" type="fixed">
+        <origin rpy="0 0 0" xyz="0 0 0"/>
+        <axis xyz="0 0 -1"/>
+        <!-- <limit effort="1000.0" lower="-1e+16" upper="1e+16" velocity="15"/> -->
+        <joint_properties damping="1" friction="1"/>
+        <parent link="base_link"/>
+        <child link="base_footprint"/>
+    </joint>
     <!-- Sensors -->
     <joint name="lidar_1_joint" type="fixed">

File: robots/mpo_700/urdf/mpo_700_body.urdf.xacro (robot description, xacro)
@@ -2,12 +2,4 @@
 <robot xmlns:xacro="http://www.ros.org/wiki/xacro" name="mpo_700">
     <link name="base_footprint"/>
-    <joint name="base_footprint_joint" type="fixed">
-        <origin rpy="0 0 0" xyz="0 0 0"/>
-        <axis xyz="0 0 -1"/>
-        <!-- <limit effort="1000.0" lower="-1e+16" upper="1e+16" velocity="15"/> -->
-        <joint_properties damping="1" friction="1"/>
-        <parent link="base_footprint"/>
-        <child link="base_link"/>
-    </joint>
     <link name="base_link">
         <inertial>
@@ -29,4 +21,12 @@
         </collision>
     </link>
+    <joint name="base_footprint_joint" type="fixed">
+        <origin rpy="0 0 0" xyz="0 0 0"/>
+        <axis xyz="0 0 -1"/>
+        <!-- <limit effort="1000.0" lower="-1e+16" upper="1e+16" velocity="15"/> -->
+        <joint_properties damping="1" friction="1"/>
+        <parent link="base_link"/>
+        <child link="base_footprint"/>
+    </joint>
     <!-- Sensors -->
     <joint name="lidar_1_joint" type="fixed">

File: robots/mpo_700/urdf/mpo_700_gazebo.urdf.xacro (robot description, xacro)
@@ -15,5 +15,5 @@
         controller_update_rate="${controller_update_rate}"
         odom_frame="odom"
-        base_frame="base_footprint"
+        base_frame="base_link"
         covariance_yaw="0.0001"
     />
