Commit message: converted all robots into modular xacros, added moveit support for ur5e and ur10 with mpo_500 and mpo_700, manually merged and resolved conflicts

File: robots/mp_400/mp_400.urdf (robot description, URDF)
Before this commit: robot mp_400, 9 links, 8 joints
Links:
- link lidar_1_link: geometry collision mesh filename=package://neo_simulation2/components/meshes/SICK-MICROSCAN3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 scale=0.001 0.001 0.001; visual mesh filename=package://neo_simulation2/components/meshes/SICK-MICROSCAN3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 scale=0.001 0.001 0.001

File: robots/mp_400/urdf/macro/mp_400_wheel_macro.xacro (robot description, xacro)
@@ -1,11 +1,12 @@
 <?xml version="1.0"?>
-<robot xmlns:xacro="http://www.ros.org/wiki/xacro" name="mpo_500">
+<robot xmlns:xacro="http://www.ros.org/wiki/xacro" name="mp_400">
     <!--WHEEL MACRO-->
-    <xacro:macro name="mpo_500_omni_wheel" params="
+    <xacro:macro name="mp_400_fixed_wheel" params="
         wheel_prefix
         parent_link
         *origin
+        meshname
         wheel_joint_type
-        has_limits
+        visual_origin_rpy
         model_scale
         ">
@@ -13,18 +14,18 @@
         <link name="${wheel_prefix}_link" type="wheel">
             <inertial>
-                <mass value="2.2"/>
+                <mass value="1.82362"/>
                 <origin rpy="0 0 0" xyz="0 0 0"/>
-                <inertia ixx="0.01" ixy="0.0" ixz="0.0" iyy="0.01" iyz="0.0" izz="0.01"/>
+                <inertia ixx="0.00399743171" ixy="0.00000004464" ixz="-0.00000002245" iyy="0.00399741733" iyz="-0.00000000164" izz="0.00739239692"/>
             </inertial>
             <visual>
-                <origin rpy="0 0 0" xyz="0 0 0"/>
+                <origin rpy="${visual_origin_rpy}" xyz="0 0 0"/>
                 <geometry>
-                    <mesh filename="package://neo_simulation2/robots/mpo_500/meshes/MPO-500-WHEEL.dae" scale="${model_scale}"/>
+                    <mesh filename="package://neo_simulation2/robots/mp_400/meshes/${meshname}.dae" scale="0.001 0.001 0.001"/>
                 </geometry>
             </visual>
             <collision>
-                <origin rpy="0 1.57 1.57" xyz="0 0 0"/>
+                <origin rpy="0 0 0" xyz="0 0 0"/>
                 <geometry>
-                    <sphere radius="0.117"/>
+                    <sphere radius="0.0765"/>
                 </geometry>
             </collision>
@@ -33,9 +34,7 @@
         <joint name="${wheel_prefix}_joint" type="${wheel_joint_type}">
             <xacro:insert_block name="origin"/>
-            <xacro:if value="${has_limits}">
-                <limit effort="1000.0" lower="-1e+16" upper="1e+16" velocity="15"/>
-            </xacro:if>
-            <axis xyz="0 1 0"/>
-            <joint_properties damping="1.0" friction="1"/>
+            <limit effort="1000.0" lower="-1e+16" upper="1e+16" velocity="3.5"/>
+            <axis xyz="-1 0 0"/>
+            <joint_properties damping="0" friction="0.0"/>
             <parent link="${parent_link}"/>
             <child link="${wheel_prefix}_link"/>

File: robots/mp_500/mp_500.urdf (robot description, URDF)
Before this commit: robot mp_500, 6 links, 5 joints
Links:
- link lidar_1_link: geometry collision mesh filename=package://neo_simulation2/components/meshes/SICK-S300.dae scale=0.001 0.001 0.001; visual mesh filename=package://neo_simulation2/components/meshes/SICK-S300.dae scale=0.001 0.001 0.001

File: robots/mp_500/urdf/macro/mp_500_wheel_macro.xacro (robot description, xacro)
@@ -1,11 +1,12 @@
 <?xml version="1.0"?>
-<robot xmlns:xacro="http://www.ros.org/wiki/xacro" name="mpo_500">
+<robot xmlns:xacro="http://www.ros.org/wiki/xacro" name="mp_500">
     <!--WHEEL MACRO-->
-    <xacro:macro name="mpo_500_omni_wheel" params="
+    <xacro:macro name="mp_500_wheel" params="
         wheel_prefix
         parent_link
+        meshname
         *origin
         wheel_joint_type
-        has_limits
+        visual_origin_rpy
         model_scale
         ">
@@ -13,18 +14,18 @@
         <link name="${wheel_prefix}_link" type="wheel">
             <inertial>
-                <mass value="2.2"/>
+                <mass value="1.82362"/>
                 <origin rpy="0 0 0" xyz="0 0 0"/>
-                <inertia ixx="0.01" ixy="0.0" ixz="0.0" iyy="0.01" iyz="0.0" izz="0.01"/>
+                <inertia ixx="0.00399743171" ixy="0.00000004464" ixz="-0.00000002245" iyy="0.00399741733" iyz="-0.00000000164" izz="0.00739239692"/>
             </inertial>
             <visual>
                 <origin rpy="0 0 0" xyz="0 0 0"/>
                 <geometry>
-                    <mesh filename="package://neo_simulation2/robots/mpo_500/meshes/MPO-500-WHEEL.dae" scale="${model_scale}"/>
+                    <mesh filename="package://neo_simulation2/robots/mp_500/meshes/${meshname}.dae" scale="0.001 0.001 0.001"/>
                 </geometry>
             </visual>
             <collision>
-                <origin rpy="0 1.57 1.57" xyz="0 0 0"/>
+                <origin rpy="0 0 0" xyz="0 0 0"/>
                 <geometry>
-                    <sphere radius="0.117"/>
+                    <mesh filename="package://neo_simulation2/robots/mp_500/meshes/${meshname}.dae" scale="0.001 0.001 0.001"/>
                 </geometry>
             </collision>
@@ -33,9 +34,7 @@
         <joint name="${wheel_prefix}_joint" type="${wheel_joint_type}">
             <xacro:insert_block name="origin"/>
-            <xacro:if value="${has_limits}">
-                <limit effort="1000.0" lower="-1e+16" upper="1e+16" velocity="15"/>
-            </xacro:if>
-            <axis xyz="0 1 0"/>
-            <joint_properties damping="1.0" friction="1"/>
+            <limit effort="1000.0" lower="-1e+16" upper="1e+16" velocity="3.5"/>
+            <axis xyz="-1 0 0"/>
+            <joint_properties damping="0" friction="0.0"/>
             <parent link="${parent_link}"/>
             <child link="${wheel_prefix}_link"/>

File: robots/mpo_700/mpo_700.urdf.xacro (robot description, xacro)
@@ -9,14 +9,6 @@
     <xacro:property name="arm" value="$(arg arm_type)"/>
     <xacro:property name="use_arm" value="false"/>
-    <!-- OmniDriveModule(ODM) joint type for both wheels and casters -->
-    <xacro:property name="ODM_joint_type" value="revolute"/>
-    <!-- When there is an arm mounted, the joints of the wheels needs
-    to be of fixed type. The reason being, both the drive modules and
-    the arm cannot publish joint states simultenously. Thus we omit
-    the visualization of the drives. Issue will be fixed, when we switch
-    to ROS 2 control. -->
-    <xacro:unless value="${arm == ''}">
-      <xacro:property name="ODM_joint_type" value="fixed"/>
-    </xacro:unless>
+    <!-- OmniDriveModule(ODM) joint type for both wheels and casters(fixed for simulation)-->
+    <xacro:property name="ODM_joint_type" value="fixed"/>
     <!-- import main body description -->
     <xacro:include filename="$(find neo_simulation2)/robots/mpo_700/urdf/mpo_700_body.urdf.xacro"/>

File: robots/mpo_700/urdf/mpo_700_body.urdf.xacro (robot description, xacro)
@@ -169,3 +169,8 @@
         <origin rpy="0 0 3.14" xyz="0.0 -0.045 -0.12"/>
     </xacro:mpo_700_wheel>
+    <!-- Import docking adapter -->
+    <xacro:include filename="$(find neo_simulation2)/robots/mpo_700/urdf/macro/docking_adapter.xacro"/>
+    <xacro:docking_adapter name="docking_adapter" parent="base_link">
+        <origin xyz="-0.300 0 0.320" rpy="0 0 -1.57" />
+    </xacro:docking_adapter>
 </robot>
