Commit message: Added UR arm support

File: robots/mpo_700/mpo_700.urdf.xacro (robot description, xacro)
@@ -6,17 +6,27 @@
     <!--set arm name to include the arm in the simulation-->
     <xacro:arg name="arm" default=""/>
-    <xacro:arg name="robot_prefix" default="mpo_700"/>
+    <!-- Model Scale -->
+    <xacro:property name="model_scale" value="0.001 0.001 0.001" />
+    <!-- Base Properties -->
+    <xacro:property name= "base_link_mass" value="140" />
+    <!-- Wheel Properties -->
+    <xacro:property name="wheel_link_mass" value="1.2" />
+    <!-- caster Wheel Properties -->
+    <xacro:property name="caster_inertial_value" value="0.27258101" />
+    <xacro:property name="caster_link_mass" value="12.7" />
+    <!-- OmniDriveModule(ODM) joint type for both wheels and casters -->
+    <xacro:property name="ODM_joint_type" value="fixed"/>
+    <!-- Arm properties-->
     <xacro:property name="arm_name" value="$(arg arm)"/>
     <xacro:property name="use_arm" value="false"/>
+    <!-- import main body description -->
+    <xacro:include filename="$(find neo_simulation2)/robots/mpo_700/urdf/mpo_700_body.urdf.xacro"/>
+    <!-- If Simulation is used -->
+    <xacro:if value="$(arg use_gazebo)">
+        <xacro:include filename="$(find neo_simulation2)/robots/mpo_700/urdf/mpo_700_gazebo.urdf.xacro"/>
+    </xacro:if>
     <!-- Check if one of the arms is used -->
     <xacro:if value="${arm_name == 'ur5' or arm_name == 'ur10' or arm_name == 'ur5e' or arm_name == 'ur10e' or arm_name == 'ec66' or arm_name == 'cs66'}">
         <xacro:property name="use_arm" value="true"/>
-    </xacro:if>
-    <xacro:include filename="$(find neo_simulation2)/robots/mpo_700/urdf/mpo_700_body.urdf.xacro"/>
-    <xacro:include filename="$(find neo_simulation2)/robots/mpo_700/urdf/mpo_700_wheel.urdf.xacro"/>
-    <xacro:include filename="$(find neo_simulation2)/robots/mpo_700/urdf/mpo_700_caster_wheel.urdf.xacro"/>
-    <!-- If Simulation is used -->
-    <xacro:if value="$(arg use_gazebo)">
-        <xacro:include filename="$(find neo_simulation2)/robots/mpo_700/urdf/mpo_700_gazebo.urdf.xacro"/>
     </xacro:if>
     <!-- If Arm is used -->
@@ -26,5 +36,5 @@
             <origin rpy="0 0 0" xyz="0.025 0 0.35"/>
             <joint_properties damping="1" friction="1"/>
-            <parent link="$(arg robot_prefix)_base_link"/>
+            <parent link="base_link"/>
             <child link="cabinet_link"/>
         </joint>
@@ -38,5 +48,5 @@
                 <origin rpy="0 0 -1.5708" xyz="0 0 0"/>
                 <geometry>
-                    <mesh filename="package://neo_simulation2/robots/mpo_700/meshes/cabin.dae" scale="0.001 0.001 0.001"/>
+                    <mesh filename="package://neo_simulation2/robots/mpo_700/meshes/cabin.dae" scale="${model_scale}"/>
                 </geometry>
             </visual>
@@ -44,12 +54,12 @@
             <origin rpy="0 0 -1.5708" xyz="0. 0. 0"/>
                 <geometry>
-                    <mesh filename="package://neo_simulation2/robots/mpo_700/meshes/cabin.dae" scale="0.001 0.001 0.001"/>
+                    <mesh filename="package://neo_simulation2/robots/mpo_700/meshes/cabin.dae" scale="${model_scale}"/>
                 </geometry>
             </collision>
         </link>
-        <!-- Universal Arms-->
+        <!-- Universal Robotics Arms-->
         <xacro:if value="${arm_name == 'ur5' or arm_name == 'ur10' or arm_name == 'ur5e' or arm_name == 'ur10e'}">
             <!-- UR arm parameters -->
-            <xacro:arg name="tf_prefix" default="" />
+            <xacro:arg name="tf_prefix" default="${arm_name}" />
             <xacro:arg name="joint_limit_params" default="$(find ur_description)/config/$(arg arm)/joint_limits.yaml"/>
             <xacro:arg name="kinematics_params" default="$(find ur_description)/config/$(arg arm)/default_kinematics.yaml"/>
@@ -65,7 +75,7 @@
             <!-- create arm -->
             <xacro:include filename="$(find ur_description)/urdf/ur_macro.xacro"/>
-            <xacro:ur_robot name="$(arg arm)"
+            <xacro:ur_robot name="${arm_name}"
                             parent="cabinet_link"
-                            tf_prefix=""
+                            tf_prefix="$(arg tf_prefix)"
                             joint_limits_parameters_file="$(arg joint_limit_params)"
                             kinematics_parameters_file="$(arg kinematics_params)"
@@ -80,5 +90,5 @@
                 <origin xyz="0.133 0.0 0.416" rpy="0.0 0.0 -1.5708" />
             </xacro:ur_robot>
-            <!-- If both Arm and Simulation is used -->
+            <!-- If both UR Arm and Simulation is used -->
             <xacro:if value="$(arg use_gazebo)">
                 <xacro:include filename="$(find ur_simulation_gazebo)/urdf/ur_gazebo.ros2_control.xacro">
@@ -103,5 +113,5 @@
         <xacro:if value="${arm_name == 'ec66' or arm_name == 'cs66'}">
         <!--Elite arm parameters-->
-        <xacro:arg name="tf_prefix" default=""/>
+        <xacro:arg name="tf_prefix" default="${arm_name}"/>
         <xacro:arg name="joint_limit_params_file" default="$(find elite_description)/config/$(arg arm)/joint_limits.yaml"/>
         <xacro:arg name="joint_origin_params_file" default="$(find elite_description)/config/$(arg arm)/joint_origins.yaml"/>
@@ -112,5 +122,5 @@
             <xacro:elite_robot
                 name="$(arg arm)"
-                tf_prefix=""
+                tf_prefix="$(arg tf_prefix)"
                 arm_parent="cabinet_link"
                 joint_limits_parameters_file="$(arg joint_limit_params_file)"
@@ -120,5 +130,5 @@
                 <origin xyz="0.133 0.0 0.416" rpy="0.0 0.0 -1.5708" />
             </xacro:elite_robot>
-            <!-- If both Arm and Simulation is used -->
+            <!-- If both Elite Arm and Simulation is used -->
             <xacro:if value="$(arg use_gazebo)">
                 <xacro:include filename="$(find elite_description)/urdf/elite_gazebo_ros2_control.urdf.xacro" />

File: robots/mpo_700/urdf/macro/mpo_700_wheel_macro.xacro (robot description, xacro)
@@ -1,20 +1,27 @@
 <?xml version="1.0"?>
 <robot xmlns:xacro="http://www.ros.org/wiki/xacro" name="mpo_700">
-    <!-- Wheel Properties -->
-    <xacro:property name="wheel_joint_type" value="fixed" />
-    <xacro:property name="wheel_joint_origin_rpy" value="0 0 0" />
-    <xacro:property name="wheel_joint_origin_xyz" value="-0.05 0. 0.18" />
-    <xacro:property name="wheel_link_mass" value="1.2" />
     <!--WHEEL MACRO-->
-    <xacro:macro name="regular_wheel" params="wheel_prefix parent ixx iyy izz has_limits">
+    <xacro:macro name="mpo_700_wheel" params="
+        wheel_prefix
+        parent_link
+        *origin
+        wheel_joint_type
+        ixx
+        iyy
+        izz
+        has_limits
+        model_scale
+        ">
+        <!--wheel joint-->
         <joint name="${wheel_prefix}_joint" type="${wheel_joint_type}">
-            <origin rpy="${wheel_joint_origin_rpy}" xyz="${wheel_joint_origin_xyz}"/>
+            <xacro:insert_block name="origin"/>
             <xacro:if value="${has_limits}">
                 <limit effort="1000.0" lower="-1e+16" upper="1e+16" velocity="15"/>
             </xacro:if>
             <axis xyz="1 0 0"/>
-            <parent link="${parent}"/>
+            <parent link="${parent_link}_link"/>
             <child link="${wheel_prefix}_link"/>
         </joint>
+        <!--wheel link-->
         <link name="${wheel_prefix}_link" type="wheel">
             <inertial>
@@ -37,8 +44,3 @@
         </link>
     </xacro:macro>
-    <!-- Wheels - Only Front wheels have limits-->
-    <xacro:regular_wheel wheel_prefix="mpo_700_wheel_front_left" ixx="0.11042056" iyy="0.11042056" izz="0.11042056" parent="mpo_700_caster_front_left_link" has_limits="true"/>
-    <xacro:regular_wheel wheel_prefix="mpo_700_wheel_front_right" ixx="0.11042056" iyy="0.11042056" izz="0.11042056" parent="mpo_700_caster_front_right_link" has_limits="true"/>
-    <xacro:regular_wheel wheel_prefix="mpo_700_wheel_back_left" ixx="0.11042056" iyy="0.11042056" izz="0.11042056" parent="mpo_700_caster_back_left_link" has_limits="false"/>
-    <xacro:regular_wheel wheel_prefix="mpo_700_wheel_back_right" ixx="0.11042056" iyy="0.11042056" izz="0.11042056" parent="mpo_700_caster_back_right_link" has_limits="false"/>
-</robot>
+   </robot>

File: robots/mpo_700/urdf/mpo_700_body.urdf.xacro (robot description, xacro)
@@ -1,6 +1,4 @@
 <?xml version="1.0"?>
 <robot xmlns:xacro="http://www.ros.org/wiki/xacro" name="mpo_700">
-    <xacro:property name="model_scale" value="0.001 0.001 0.001" />
-    <xacro:property name= "base_link_mass" value="140" />
     <link name="base_footprint"/>
     <joint name="base_footprint_joint" type="fixed">
@@ -10,7 +8,7 @@
         <joint_properties damping="1" friction="1"/>
         <parent link="base_footprint"/>
-        <child link="$(arg robot_prefix)_base_link"/>
+        <child link="base_link"/>
     </joint>
-    <link name="$(arg robot_prefix)_base_link">
+    <link name="base_link">
         <inertial>
             <mass value="${base_link_mass}"/>
@@ -35,5 +33,5 @@
         <axis xyz="0 1 0"/>
         <origin rpy="3.14 0 0.79" xyz="0.338 0.288 0.223"/>
-        <parent link="$(arg robot_prefix)_base_link"/>
+        <parent link="base_link"/>
         <child link="lidar_1_link"/>
     </joint>
@@ -60,5 +58,5 @@
         <axis xyz="0 1 0"/>
         <origin rpy="3.14 0 3.93" xyz="-0.338 -0.288 0.223"/>
-        <parent link="$(arg robot_prefix)_base_link"/>
+        <parent link="base_link"/>
         <child link="lidar_2_link"/>
     </joint>
@@ -82,3 +80,100 @@
         </collision>
     </link>
+    <!-- Import wheel macros -->
+    <xacro:include filename="$(find neo_simulation2)/robots/mpo_700/urdf/macro/mpo_700_wheel_macro.xacro"/>
+    <xacro:include filename="$(find neo_simulation2)/robots/mpo_700/urdf/macro/mpo_700_caster_wheel_macro.xacro"/>
+    <!-- Caster wheels -->
+    <xacro:mpo_700_caster_wheel
+        caster_prefix="caster_front_left"
+        caster_joint_type="${ODM_joint_type}"
+        parent_link="base_link"
+        caster_inertial_value="${caster_inertial_value}"
+        caster_link_mass="${caster_link_mass}"
+        has_limits="false"
+        model_scale="${model_scale}"
+        >
+        <origin xyz="0.24 0.18 0.27" rpy="3.14 0 -1.57"/>
+    </xacro:mpo_700_caster_wheel>
+    <xacro:mpo_700_caster_wheel
+        caster_prefix="caster_front_right"
+        caster_joint_type="${ODM_joint_type}"
+        parent_link="base_link"
+        caster_inertial_value="${caster_inertial_value}"
+        caster_link_mass="${caster_link_mass}"
+        has_limits="false"
+        model_scale="${model_scale}"
+        >
+        <origin xyz="-0.24 -0.18 0.27" rpy="3.14 0 1.57"/>
+    </xacro:mpo_700_caster_wheel>
+    <xacro:mpo_700_caster_wheel
+        caster_prefix="caster_back_left"
+        caster_joint_type="${ODM_joint_type}"
+        parent_link="base_link"
+        caster_inertial_value="${caster_inertial_value}"
+        caster_link_mass="${caster_link_mass}"
+        has_limits="false"
+        model_scale="${model_scale}"
+        >
+        <origin xyz="0.24 -0.18 0.27" rpy="3.14 0 1.57"/>
+    </xacro:mpo_700_caster_wheel>
+    <xacro:mpo_700_caster_wheel
+        caster_prefix="caster_back_right"
+        caster_joint_type="${ODM_joint_type}"
+        parent_link="base_link"
+        caster_inertial_value="${caster_inertial_value}"
+        caster_link_mass="${caster_link_mass}"
+        has_limits="false"
+        model_scale="${model_scale}"
+        >
+        <origin xyz="-0.24 0.18 0.27" rpy="3.14 0 -1.57"/>
+    </xacro:mpo_700_caster_wheel>
+    <!-- NOTE: Only Front wheels have limits-->
+    <xacro:mpo_700_wheel
+        wheel_prefix="wheel_front_left"
+        parent_link="caster_front_left"
+        wheel_joint_type="${ODM_joint_type}"
+        ixx="0.11042056"
+        iyy="0.11042056"
+        izz="0.11042056"
+        has_limits="true"
+        model_scale="${model_scale}"
+        >
+        <origin xyz="-0.05 0. 0.18" rpy="0 0 0"/>
+    </xacro:mpo_700_wheel>
+    <xacro:mpo_700_wheel
+        wheel_prefix="wheel_front_right"
+        parent_link="caster_front_right"
+        wheel_joint_type="${ODM_joint_type}"
+        ixx="0.11042056"
+        iyy="0.11042056"
+        izz="0.11042056"
+        has_limits="true"
+        model_scale="${model_scale}"
+        >
+        <origin xyz="-0.05 0. 0.18" rpy="0 0 0"/>
+    </xacro:mpo_700_wheel>
+    <xacro:mpo_700_wheel
+        wheel_prefix="wheel_back_left"
+        parent_link="caster_back_left"
+        wheel_joint_type="${ODM_joint_type}"
+        ixx="0.11042056"
+        iyy="0.11042056"
+        izz="0.11042056"
+        has_limits="false"
+        model_scale="${model_scale}"
+        >
+        <origin xyz="-0.05 0. 0.18" rpy="0 0 0"/>
+    </xacro:mpo_700_wheel>
+    <xacro:mpo_700_wheel
+        wheel_prefix="wheel_back_right"
+        parent_link="caster_back_right"
+        wheel_joint_type="${ODM_joint_type}"
+        ixx="0.11042056"
+        iyy="0.11042056"
+        izz="0.11042056"
+        has_limits="false"
+        model_scale="${model_scale}"
+        >
+        <origin xyz="-0.05 0. 0.18" rpy="0 0 0"/>
+    </xacro:mpo_700_wheel>
 </robot>

File: robots/mpo_700/urdf/mpo_700_gazebo.urdf.xacro (robot description, xacro)
@@ -1,126 +1,70 @@
 <?xml version="1.0"?>
 <robot xmlns:xacro="http://www.ros.org/wiki/xacro" name="mpo_700">
+    <!-- Include macros -->
+    <xacro:include filename="$(find neo_simulation2)/robots/mpo_700/urdf/macro/gazebo_lidar_macro.xacro" />
+    <xacro:include filename="$(find neo_simulation2)/robots/mpo_700/urdf/macro/gazebo_mpo_700_wheel_macro.xacro" />
+    <xacro:include filename="$(find neo_simulation2)/robots/mpo_700/urdf/macro/gazebo_object_controller_macro.xacro" />
+    <!-- Properties -->
     <xacro:property name="wheel_mu" value="0.0001" />
-    <xacro:property name="lidar_resolution" value="0.05" />
-    <!--Gazebo Wheel Macro-->
-    <xacro:macro name="wheel_gazebo" params="wheel_link">
-        <gazebo reference="${wheel_link}">
-            <!-- <kp> 10000 </kp> -->
-            <!-- <fdir1>0 1 0</fdir1> -->
-            <!-- <slip1> 0.1 </slip1> -->
-            <mu1>${wheel_mu}</mu1>
-            <mu2>${wheel_mu}</mu2>
-        </gazebo>
-    </xacro:macro>
-      <!-- SENSORS -->
-      <!-- Sick S300 - Comment/Uncomment if required -->
-      <!-- <xacro:include filename="$(find neo_simulation2)/robots/mpo_700/xacros/sick_S300.xacro" /> -->
-      <!--Ultrasonics, cameras and IMU's  -->
-      <gazebo reference="lidar_1_link">
-          <sensor name="lidar_1_sensor" type="ray">
-              <always_on>true</always_on>
-              <pose>0 0 0 0 0 0</pose>
-              <visualize>false</visualize>
-              <update_rate>40</update_rate>
-              <ray>
-                  <scan>
-                      <horizontal>
-                          <samples>720</samples>
-                          <resolution>1</resolution>
-                          <min_angle>-1.48</min_angle>
-                          <max_angle>1.48</max_angle>
-                      </horizontal>
-                  </scan>
-                  <range>
-                      <min>0.10</min>
-                      <max>30.0</max>
-                      <resolution>${lidar_resolution}</resolution>
-                  </range>
-                  <noise>
-                      <type>gaussian</type>
-                      <!-- Noise parameters based on published spec for Hokuyo laser
-                              achieving "+-30mm" accuracy at range < 10m.  A mean of 0.0m and
-                              stddev of 0.01m will put 99.7% of samples within 0.03m of the true
-                              reading. -->
-                      <mean>0.0</mean>
-                      <stddev>0.01</stddev>
-                  </noise>
-              </ray>
-              <plugin filename="libgazebo_ros_ray_sensor.so" name="lidar_1">
-                  <ros>
-                      <!-- <namespace>   </namespace> -->
-                      <argument>~/out:=scan</argument>
-                  </ros>
-                  <!-- Set output to sensor_msgs/LaserScan to get same output type as gazebo_ros_laser -->
-                  <output_type>sensor_msgs/LaserScan</output_type>
-                  <frame_name>lidar_1_link</frame_name>
-              </plugin>
-          </sensor>
-      </gazebo>
-      <gazebo reference="lidar_2_link">
-          <sensor name="lidar_2_sensor" type="ray">
-              <pose>0 0 0 0 0 0</pose>
-              <visualize>false</visualize>
-              <update_rate>40</update_rate>
-                  <ray>
-                      <scan>
-                          <horizontal>
-                              <samples>720</samples>
-                              <resolution>1</resolution>
-                              <min_angle>-1.48</min_angle>
-                              <max_angle>1.48</max_angle>
-                          </horizontal>
-                      </scan>
-                      <range>
-                          <min>0.10</min>
-                          <max>30.0</max>
-                          <resolution>${lidar_resolution}</resolution>
-                      </range>
-                      <noise>
-                          <type>gaussian</type>
-                          <!-- Noise parameters based on published spec for Hokuyo laser
-                                  achieving "+-30mm" accuracy at range < 10m.  A mean of 0.0m and
-                                  stddev of 0.01m will put 99.7% of samples within 0.03m of the true
-                                  reading. -->
-                          <mean>0.0</mean>
-                          <stddev>0.01</stddev>
-                      </noise>
-                  </ray>
-              <plugin filename="libgazebo_ros_ray_sensor.so" name="lidar_2">
-                  <ros>
-                    <!-- <namespace> </namespace> -->
-                      <argument>~/out:=scan2</argument>
-                  </ros>
-                  <!-- Set output to sensor_msgs/LaserScan to get same output type as gazebo_ros_laser -->
-                  <output_type>sensor_msgs/LaserScan</output_type>
-                  <frame_name>lidar_2_link</frame_name>
-              </plugin>
-          </sensor>
-      </gazebo>
-      <gazebo>
-          <plugin name="object_controller" filename="libgazebo_ros_planar_move.so">
-              <commandTopic>cmd_vel</commandTopic>
-              <odometryTopic>odom</odometryTopic>
-              <robotNamespace><remapping>/tf:=tf</remapping>  </robotNamespace>
-              <ros>    <remapping>/tf:=tf</remapping>    </ros>
-              <!-- Set control loop update rate -->
-              <odometryRate>100</odometryRate>
-              <!-- Set odom publish rate -->
-              <publish_rate>100</publish_rate>
-              <!-- Set if odom required -->
-              <publish_odom>true</publish_odom>
-              <publish_odom_tf>true</publish_odom_tf>
-              <!-- Frame IDs -->
-              <odometryFrame>odom</odometryFrame>
-              <robotBaseFrame>base_foot</robotBaseFrame>
-              <!-- Set odom covariance -->
-              <covariance_x>0.0001</covariance_x>
-              <covariance_y>0.0001</covariance_y>
-              <covariance_yaw>0.0001</covariance_yaw>
-          </plugin>
-      </gazebo>
-    <xacro:wheel_gazebo wheel_link="mpo_700_wheel_front_right_link" />
-    <xacro:wheel_gazebo wheel_link="mpo_700_wheel_back_right_link" />
-    <xacro:wheel_gazebo wheel_link="mpo_700_wheel_front_left_link" />
-    <xacro:wheel_gazebo wheel_link="mpo_700_wheel_back_left_link" />
+    <xacro:property name="lidar_1_update_rate" value="40" />
+    <xacro:property name="lidar_2_update_rate" value="40" />
+    <xacro:property name="controller_update_rate" value="100" />
+    <xacro:property name="odom_update_rate" value="100" />
+    <!--Object Controller-->
+    <xacro:gazebo_object_controller
+        odom_update_rate="${odom_update_rate}"
+        controller_update_rate="${controller_update_rate}"
+        odom_frame="odom"
+        base_frame="base_footprint"
+    />
+    <!--Lidar Sensors-->
+    <xacro:gazebo_lidar_sensor
+        sensor_name="lidar_1_sensor"
+        link_name="lidar_1_link"
+        update_rate="${lidar_1_update_rate}"
+        min_range="0.10"
+        max_range="30.0"
+        horizontal_samples="720"
+        min_angle="-1.48"
+        max_angle="1.48"
+        noise_mean="0.0"
+        noise_stddev="0.01"
+        topic_name="scan"
+        visualize="false"
+    />
+    <xacro:gazebo_lidar_sensor
+        sensor_name="lidar_2_sensor"
+        link_name="lidar_2_link"
+        update_rate="${lidar_2_update_rate}"
+        min_range="0.10"
+        max_range="30.0"
+        horizontal_samples="720"
+        min_angle="-1.48"
+        max_angle="1.48"
+        noise_mean="0.0"
+        noise_stddev="0.01"
+        topic_name="scan2"
+        visualize="false"
+    />
+    <!--Wheels-->
+    <xacro:gazebo_mpo_700_wheel
+        wheel_prefix="wheel_front_right"
+        wheel_mu="${wheel_mu}"
+        />
+    <xacro:gazebo_mpo_700_wheel
+        wheel_prefix="wheel_back_right"
+        wheel_mu="${wheel_mu}"
+        />
+    <xacro:gazebo_mpo_700_wheel
+        wheel_prefix="wheel_front_left"
+        wheel_mu="${wheel_mu}"
+        />
+    <xacro:gazebo_mpo_700_wheel
+        wheel_prefix="wheel_back_left"
+        wheel_mu="${wheel_mu}"
+        />
+    <!-- SENSORS -->
+    <!-- Sick S300 - Comment/Uncomment if required -->
+    <!-- <xacro:include filename="$(find neo_simulation2)/robots/mpo_700/xacros/sick_S300.xacro" /> -->
+    <!--Ultrasonics, cameras and IMU's  -->
 </robot>
