Commit message: updates to urdf, replaced old castor and wheel models with new ones from mpo-700-2 package, restructured files, added robot prefix to ur controller (ur10, ur10e,ur5,ur5e) - hardcoded for now, added common initial joint positions for all ur arms

File: robots/mpo_700/mpo_700.urdf.xacro (robot description, xacro)
@@ -5,5 +5,5 @@
     <xacro:arg name="use_gazebo" default="true"/>
     <!--set arm name to include the arm in the simulation-->
-    <xacro:arg name="arm" default=""/>
+    <xacro:arg name="arm_type" default=""/>
     <!-- Model Scale -->
     <xacro:property name="model_scale" value="0.001 0.001 0.001" />
@@ -15,9 +15,17 @@
     <xacro:property name="caster_inertial_value" value="0.27258101" />
     <xacro:property name="caster_link_mass" value="12.7" />
+    <!-- Arm properties-->
+    <xacro:property name="arm" value="$(arg arm_type)"/>
+    <xacro:property name="use_arm" value="false"/>
     <!-- OmniDriveModule(ODM) joint type for both wheels and casters -->
-    <xacro:property name="ODM_joint_type" value="fixed"/>
-    <!-- Arm properties-->
-    <xacro:property name="arm_name" value="$(arg arm)"/>
-    <xacro:property name="use_arm" value="false"/>
+    <xacro:property name="ODM_joint_type" value="revolute"/>
+    <!-- When there is an arm mounted, the joints of the wheels needs
+    to be of fixed type. The reason being, both the drive modules and
+    the arm cannot publish joint states simultenously. Thus we omit
+    the visualization of the drives. Issue will be fixed, when we switch
+    to ROS 2 control. -->
+    <xacro:unless value="${arm == ''}">
+      <xacro:property name="ODM_joint_type" value="fixed"/>
+    </xacro:unless>
     <!-- import main body description -->
     <xacro:include filename="$(find neo_simulation2)/robots/mpo_700/urdf/mpo_700_body.urdf.xacro"/>
@@ -27,5 +35,5 @@
     </xacro:if>
     <!-- Check if one of the arms is used -->
-    <xacro:if value="${arm_name == 'ur5' or arm_name == 'ur10' or arm_name == 'ur5e' or arm_name == 'ur10e' or arm_name == 'ec66' or arm_name == 'cs66'}">
+    <xacro:if value="${arm == 'ur5' or arm == 'ur10' or arm == 'ur5e' or arm == 'ur10e' or arm == 'ec66' or arm == 'cs66'}">
         <xacro:property name="use_arm" value="true"/>
     </xacro:if>
@@ -59,23 +67,28 @@
         </link>
         <!-- Universal Robotics Arms-->
-        <xacro:if value="${arm_name == 'ur5' or arm_name == 'ur10' or arm_name == 'ur5e' or arm_name == 'ur10e'}">
+        <xacro:if value="${arm == 'ur5' or arm == 'ur10' or arm == 'ur5e' or arm == 'ur10e'}">
+            <!-- create arm from macro-->
+            <xacro:include filename="$(find ur_description)/urdf/ur_macro.xacro"/>
             <!-- UR arm parameters -->
-            <xacro:arg name="tf_prefix" default="${arm_name}" />
-            <xacro:arg name="joint_limit_params" default="$(find ur_description)/config/$(arg arm)/joint_limits.yaml"/>
-            <xacro:arg name="kinematics_params" default="$(find ur_description)/config/$(arg arm)/default_kinematics.yaml"/>
-            <xacro:arg name="physical_params" default="$(find ur_description)/config/$(arg arm)/physical_parameters.yaml"/>
-            <xacro:arg name="visual_params" default="$(find ur_description)/config/$(arg arm)/visual_parameters.yaml"/>
+            <xacro:arg name="tf_prefix" default="${arm}" />
+            <xacro:arg name="joint_limit_params" default="$(find ur_description)/config/$(arg arm_type)/joint_limits.yaml"/>
+            <xacro:arg name="kinematics_params" default="$(find ur_description)/config/$(arg arm_type)/default_kinematics.yaml"/>
+            <xacro:arg name="physical_params" default="$(find ur_description)/config/$(arg arm_type)/physical_parameters.yaml"/>
+            <xacro:arg name="visual_params" default="$(find ur_description)/config/$(arg arm_type)/visual_parameters.yaml"/>
             <xacro:arg name="transmission_hw_interface" default="hardware_interface/PositionJointInterface"/>
             <xacro:arg name="safety_limits" default="false"/>
             <xacro:arg name="safety_pos_margin" default="0.15"/>
             <xacro:arg name="safety_k_position" default="20"/>
-            <xacro:arg name="force_abs_paths" default="true" />
-            <xacro:arg name="simulation_controllers" default="$(find ur_simulation_gazebo)/config/ur_controllers.yaml" />
-            <xacro:arg name="initial_joint_positions_file" default="$(find ur_description)/config/initial_positions.yaml"/>
-            <!-- create arm -->
-            <xacro:include filename="$(find ur_description)/urdf/ur_macro.xacro"/>
-            <xacro:ur_robot name="${arm_name}"
+            <xacro:arg name="sim_gazebo" default="$(arg use_gazebo)" />
+            <xacro:arg name="simulation_controllers" default="$(find neo_simulation2)/configs/ur_config/$(arg arm_type)/ur_controllers.yaml"/>
+            <xacro:arg name="initial_positions_file" default="$(find neo_simulation2)/configs/ur_config/initial_joint_positions.yaml"/>
+            <!-- parse initial positions as a dictionary -->
+            <xacro:property
+                name="ur_initial_positions"
+                value="${xacro.load_yaml('$(arg initial_positions_file)')}"
+                />
+            <xacro:ur_robot name="${arm}"
+                            tf_prefix="$(arg tf_prefix)"
                             parent="cabinet_link"
-                            tf_prefix="$(arg tf_prefix)"
                             joint_limits_parameters_file="$(arg joint_limit_params)"
                             kinematics_parameters_file="$(arg kinematics_params)"
@@ -85,5 +98,6 @@
                             safety_pos_margin="$(arg safety_pos_margin)"
                             safety_k_position="$(arg safety_k_position)"
-                            force_abs_paths="$(arg force_abs_paths)"
+                            sim_gazebo="$(arg sim_gazebo)"
+                            initial_positions = "${ur_initial_positions}"
                             >
                 <!-- position robot in the world -->
@@ -91,9 +105,7 @@
             </xacro:ur_robot>
             <!-- If both UR Arm and Simulation is used -->
-            <xacro:if value="$(arg use_gazebo)">
-                <xacro:include filename="$(find ur_simulation_gazebo)/urdf/ur_gazebo.ros2_control.xacro">
-                    <parameters>$(arg simulation_controllers)</parameters>
-                </xacro:include>
-                <gazebo reference="cabinet_link"></gazebo>
+            <xacro:if value="$(arg sim_gazebo)">
+                <gazebo reference="cabinet_link">
+                </gazebo>
                 <gazebo>
                     <plugin filename="libgazebo_ros2_control.so" name="gazebo_ros2_control">
@@ -101,25 +113,18 @@
                     </plugin>
                 </gazebo>
-                <!-- ros2 control instance -->
-                <xacro:ur_ros2_control
-                    name="$(arg arm)"
-                    tf_prefix="$(arg tf_prefix)"
-                    transmission_hw_interface="$(arg transmission_hw_interface)"
-                    initial_positions="${xacro.load_yaml('$(arg initial_joint_positions_file)')}"
-                />
             </xacro:if>
         </xacro:if>
         <!-- Elite Arm -->
-        <xacro:if value="${arm_name == 'ec66' or arm_name == 'cs66'}">
+        <xacro:if value="${arm == 'ec66' or arm == 'cs66'}">
         <!--Elite arm parameters-->
-        <xacro:arg name="tf_prefix" default="${arm_name}"/>
-        <xacro:arg name="joint_limit_params_file" default="$(find elite_description)/config/$(arg arm)/joint_limits.yaml"/>
-        <xacro:arg name="joint_origin_params_file" default="$(find elite_description)/config/$(arg arm)/joint_origins.yaml"/>
-        <xacro:arg name="link_inertials_params_file" default="$(find elite_description)/config/$(arg arm)/link_inertials.yaml"/>
-        <xacro:arg name="initial_joint_positions_file" default="$(find elite_description)/config/$(arg arm)/initial_positions.yaml"/>
+        <xacro:arg name="tf_prefix" default="${arm}"/>
+        <xacro:arg name="joint_limit_params_file" default="$(find elite_description)/config/$(arg arm_type)/joint_limits.yaml"/>
+        <xacro:arg name="joint_origin_params_file" default="$(find elite_description)/config/$(arg arm_type)/joint_origins.yaml"/>
+        <xacro:arg name="link_inertials_params_file" default="$(find elite_description)/config/$(arg arm_type)/link_inertials.yaml"/>
+        <xacro:arg name="initial_joint_positions_file" default="$(find elite_description)/config/$(arg arm_type)/initial_positions.yaml"/>
             <!-- create arm -->
             <xacro:include filename="$(find elite_description)/urdf/macro/elite_macro.xacro" />
             <xacro:elite_robot
-                name="$(arg arm)"
+                name="$(arg arm_type)"
                 tf_prefix="$(arg tf_prefix)"
                 arm_parent="cabinet_link"

File: robots/mpo_700/urdf/macro/mpo_700_caster_wheel_macro.xacro (robot description, xacro)
@@ -5,4 +5,5 @@
         caster_prefix
         caster_joint_type
+        link_origin_rpy
         *origin
         parent_link
@@ -19,5 +20,5 @@
             </inertial>
             <visual>
-                <origin xyz="0 0 0.10" rpy="0 0 0"/>
+                <origin xyz="0 0 0" rpy="${link_origin_rpy}"/>
                 <geometry>
                     <mesh filename="package://neo_simulation2/robots/mpo_700/meshes/MPO-700-HEAD.dae" scale="${model_scale}"/>
@@ -25,5 +26,5 @@
             </visual>
             <collision>
-                <origin xyz="0 0 0.10" rpy="0 0 0"/>
+                <origin xyz="0 0 0" rpy="${link_origin_rpy}"/>
                 <geometry>
                     <mesh filename="package://neo_simulation2/robots/mpo_700/meshes/MPO-700-HEAD.dae" scale="${model_scale}"/>
@@ -33,9 +34,9 @@
         <joint name="${caster_prefix}_joint" type="${caster_joint_type}">
             <xacro:insert_block name="origin"/>
-            <axis xyz="0 0 -1"/>
+            <axis xyz="0 0 1"/>
             <xacro:if value="${has_limits}">
-                <limit effort="1000.0" lower="-1e+16" upper="1e+16" velocity="15"/>
+                <limit effort="1000.0" lower="-1e+16" upper="1e+16" velocity="6.5"/>
             </xacro:if>
-            <joint_properties damping="1" friction="1"/>
+            <joint_properties damping="30" friction="110"/>
             <parent link="${parent_link}"/>
             <child link="${caster_prefix}_link"/>

File: robots/mpo_700/urdf/macro/mpo_700_wheel_macro.xacro (robot description, xacro)
@@ -5,4 +5,5 @@
         wheel_prefix
         parent_link
+        link_origin_rpy
         *origin
         wheel_joint_type
@@ -13,14 +14,4 @@
         model_scale
         ">
-        <!--wheel joint-->
-        <joint name="${wheel_prefix}_joint" type="${wheel_joint_type}">
-            <xacro:insert_block name="origin"/>
-            <xacro:if value="${has_limits}">
-                <limit effort="1000.0" lower="-1e+16" upper="1e+16" velocity="15"/>
-            </xacro:if>
-            <axis xyz="1 0 0"/>
-            <parent link="${parent_link}_link"/>
-            <child link="${wheel_prefix}_link"/>
-        </joint>
         <!--wheel link-->
         <link name="${wheel_prefix}_link" type="wheel">
@@ -31,5 +22,5 @@
             </inertial>
             <visual>
-                <origin rpy="0 0 0" xyz="0 0 0"/>
+                <origin rpy="${link_origin_rpy}" xyz="0 0 0"/>
                 <geometry>
                     <mesh filename="package://neo_simulation2/robots/mpo_700/meshes/MPO-700-WHEEL.dae" scale="${model_scale}"/>
@@ -39,8 +30,20 @@
                 <origin rpy="0 0 0" xyz="0 0 0"/>
                 <geometry>
-                    <mesh filename="package://neo_simulation2/robots/mpo_700/meshes/MPO-700-WHEEL.dae" scale="${model_scale}"/>
+                    <sphere radius="0.09"/>
+                    <!-- <mesh filename="package://neo_simulation2/robots/mpo_700/meshes/MPO-700-WHEEL.dae" scale="${model_scale}"/> -->
                 </geometry>
             </collision>
         </link>
+        <!--wheel joint-->
+        <joint name="${wheel_prefix}_joint" type="${wheel_joint_type}">
+            <xacro:insert_block name="origin"/>
+            <xacro:if value="${has_limits}">
+                <limit effort="1000.0" lower="-1e+16" upper="1e+16" velocity="20.5"/>
+            </xacro:if>
+            <axis xyz="0 -1 0"/>
+            <joint_properties damping="30" friction="110"/>
+            <parent link="${parent_link}_link"/>
+            <child link="${wheel_prefix}_link"/>
+        </joint>
     </xacro:macro>
    </robot>

File: robots/mpo_700/urdf/mpo_700_body.urdf.xacro (robot description, xacro)
@@ -87,50 +87,55 @@
         caster_prefix="caster_front_left"
         caster_joint_type="${ODM_joint_type}"
+        link_origin_rpy="0 0 0"
         parent_link="base_link"
         caster_inertial_value="${caster_inertial_value}"
         caster_link_mass="${caster_link_mass}"
-        has_limits="false"
+        has_limits="true"
         model_scale="${model_scale}"
         >
-        <origin xyz="0.24 0.18 0.27" rpy="3.14 0 -1.57"/>
+        <origin rpy="0 0 0" xyz="0.24 0.18 0.22"/>
     </xacro:mpo_700_caster_wheel>
     <xacro:mpo_700_caster_wheel
         caster_prefix="caster_front_right"
         caster_joint_type="${ODM_joint_type}"
+        link_origin_rpy="0 0 3.14"
         parent_link="base_link"
         caster_inertial_value="${caster_inertial_value}"
         caster_link_mass="${caster_link_mass}"
-        has_limits="false"
+        has_limits="true"
         model_scale="${model_scale}"
         >
-        <origin xyz="-0.24 -0.18 0.27" rpy="3.14 0 1.57"/>
+        <origin rpy="0 0 0" xyz="0.24 -0.18 0.22"/>
     </xacro:mpo_700_caster_wheel>
     <xacro:mpo_700_caster_wheel
         caster_prefix="caster_back_left"
         caster_joint_type="${ODM_joint_type}"
+        link_origin_rpy="0 0 0"
         parent_link="base_link"
         caster_inertial_value="${caster_inertial_value}"
         caster_link_mass="${caster_link_mass}"
-        has_limits="false"
+        has_limits="true"
         model_scale="${model_scale}"
         >
-        <origin xyz="0.24 -0.18 0.27" rpy="3.14 0 1.57"/>
+        <origin rpy="0 0 0" xyz="-0.24 0.18 0.22"/>
     </xacro:mpo_700_caster_wheel>
     <xacro:mpo_700_caster_wheel
         caster_prefix="caster_back_right"
         caster_joint_type="${ODM_joint_type}"
+        link_origin_rpy="0 0 3.14"
         parent_link="base_link"
         caster_inertial_value="${caster_inertial_value}"
         caster_link_mass="${caster_link_mass}"
-        has_limits="false"
+        has_limits="true"
         model_scale="${model_scale}"
         >
-        <origin xyz="-0.24 0.18 0.27" rpy="3.14 0 -1.57"/>
+        <origin rpy="0 0 0" xyz="-0.24 -0.18 0.22"/>
     </xacro:mpo_700_caster_wheel>
-    <!-- NOTE: Only Front wheels have limits-->
+    <!-- NOTE: All wheels have limits-->
     <xacro:mpo_700_wheel
         wheel_prefix="wheel_front_left"
         parent_link="caster_front_left"
         wheel_joint_type="${ODM_joint_type}"
+        link_origin_rpy="0 0 3.14"
         ixx="0.11042056"
         iyy="0.11042056"
@@ -139,5 +144,5 @@
         model_scale="${model_scale}"
         >
-        <origin xyz="-0.05 0. 0.18" rpy="0 0 0"/>
+        <origin rpy="0 0 0" xyz="0.0 0.045 -0.12"/>
     </xacro:mpo_700_wheel>
     <xacro:mpo_700_wheel
@@ -145,4 +150,5 @@
         parent_link="caster_front_right"
         wheel_joint_type="${ODM_joint_type}"
+        link_origin_rpy="0 0 3.14"
         ixx="0.11042056"
         iyy="0.11042056"
@@ -151,5 +157,5 @@
         model_scale="${model_scale}"
         >
-        <origin xyz="-0.05 0. 0.18" rpy="0 0 0"/>
+        <origin rpy="0 0 3.14" xyz="0.0 -0.045 -0.12"/>
     </xacro:mpo_700_wheel>
     <xacro:mpo_700_wheel
@@ -157,11 +163,12 @@
         parent_link="caster_back_left"
         wheel_joint_type="${ODM_joint_type}"
+        link_origin_rpy="0 0 3.14"
         ixx="0.11042056"
         iyy="0.11042056"
         izz="0.11042056"
-        has_limits="false"
+        has_limits="true"
         model_scale="${model_scale}"
         >
-        <origin xyz="-0.05 0. 0.18" rpy="0 0 0"/>
+        <origin rpy="0 0 0" xyz="0.0 0.045 -0.12"/>
     </xacro:mpo_700_wheel>
     <xacro:mpo_700_wheel
@@ -169,11 +176,12 @@
         parent_link="caster_back_right"
         wheel_joint_type="${ODM_joint_type}"
+        link_origin_rpy="0 0 3.14"
         ixx="0.11042056"
         iyy="0.11042056"
         izz="0.11042056"
-        has_limits="false"
+        has_limits="true"
         model_scale="${model_scale}"
         >
-        <origin xyz="-0.05 0. 0.18" rpy="0 0 0"/>
+        <origin rpy="0 0 3.14" xyz="0.0 -0.045 -0.12"/>
     </xacro:mpo_700_wheel>
 </robot>

Commit message: Added launch argument to include docking adapter(True for MPO-700 only)

File: robots/mpo_700/mpo_700.urdf.xacro (robot description, xacro)
@@ -4,4 +4,6 @@
     <!--set use_gazebo = false for implementation on real robot-->
     <xacro:arg name="use_gazebo" default="true"/>
+    <!--set use_docking_adapter = true to use adapter with the robot-->
+    <xacro:arg name="use_docking_adapter" default="false"/>
     <!--set arm name to include the arm in the simulation-->
     <xacro:arg name="arm_type" default=""/>

File: robots/mpo_700/urdf/mpo_700_body.urdf.xacro (robot description, xacro)
@@ -170,7 +170,9 @@
     </xacro:mpo_700_wheel>
     <!-- Import docking adapter -->
-    <xacro:include filename="$(find neo_simulation2)/robots/mpo_700/urdf/macro/docking_adapter.xacro"/>
-    <xacro:docking_adapter name="docking_adapter" parent="base_link">
-        <origin xyz="-0.300 0 0.320" rpy="0 0 -1.57" />
-    </xacro:docking_adapter>
+    <xacro:if value="$(arg use_docking_adapter)">
+        <xacro:include filename="$(find neo_simulation2)/robots/mpo_700/urdf/macro/docking_adapter.xacro"/>
+        <xacro:docking_adapter name="docking_adapter" parent="base_link">
+            <origin xyz="-0.300 0 0.320" rpy="0 0 -1.57" />
+        </xacro:docking_adapter>
+    </xacro:if>
 </robot>
