Commit message: Updated mp_500 and mp_400 urdf

File: robots/mp_400/urdf/mp_400_body.urdf.xacro (robot description, xacro)
@@ -2,12 +2,4 @@
 <robot xmlns:xacro="http://www.ros.org/wiki/xacro" name="mp_400">
     <link name="base_footprint"/>
-    <joint name="base_footprint_joint" type="fixed">
-        <origin rpy="0 0 0" xyz="0 0 0"/>
-        <axis xyz="0 0 -1"/>
-        <!-- <limit effort="1000.0" lower="-1e+16" upper="1e+16" velocity="3.5"/> -->
-        <joint_properties damping="1" friction="1"/>
-        <parent link="base_footprint"/>
-        <child link="base_link"/>
-    </joint>
     <link name="base_link">
         <inertial>
@@ -29,4 +21,12 @@
         </collision>
     </link>
+    <joint name="base_footprint_joint" type="fixed">
+        <origin rpy="0 0 0" xyz="0 0 0"/>
+        <axis xyz="0 0 -1"/>
+        <!-- <limit effort="1000.0" lower="-1e+16" upper="1e+16" velocity="3.5"/> -->
+        <joint_properties damping="1" friction="1"/>
+        <parent link="base_link"/>
+        <child link="base_footprint"/>
+    </joint>
     <!-- Sensors -->
     <joint name="lidar_1_joint" type="fixed">

File: robots/mp_400/urdf/mp_400_gazebo.urdf.xacro (robot description, xacro)
@@ -27,5 +27,5 @@
         odometry_topic="odom"
         odom_frame="odom"
-        base_frame="base_footprint"
+        base_frame="base_link"
         max_wheel_torque="1000"
         max_acceleration="20.0"

File: robots/mp_500/urdf/mp_500_body.urdf.xacro (robot description, xacro)
@@ -2,12 +2,4 @@
 <robot xmlns:xacro="http://www.ros.org/wiki/xacro" name="mp_500">
     <link name="base_footprint"/>
-    <joint name="base_footprint_joint" type="fixed">
-        <origin rpy="0 0 0" xyz="0 0 0"/>
-        <axis xyz="0 0 -1"/>
-        <!-- <limit effort="1000.0" lower="-1e+16" upper="1e+16" velocity="3.5"/> -->
-        <joint_properties damping="1" friction="1"/>
-        <parent link="base_footprint"/>
-        <child link="base_link"/>
-    </joint>
     <link name="base_link">
         <inertial>
@@ -29,4 +21,12 @@
         </collision>
     </link>
+    <joint name="base_footprint_joint" type="fixed">
+        <origin rpy="0 0 0" xyz="0 0 0"/>
+        <axis xyz="0 0 -1"/>
+        <!-- <limit effort="1000.0" lower="-1e+16" upper="1e+16" velocity="3.5"/> -->
+        <joint_properties damping="1" friction="1"/>
+        <parent link="base_link"/>
+        <child link="base_footprint"/>
+    </joint>
     <joint name="caster_wheel_joint" type="fixed">
         <origin rpy="-1.570796 0 1.570796 " xyz="-0.43 0. 0.176"/>

File: robots/mp_500/urdf/mp_500_gazebo.urdf.xacro (robot description, xacro)
@@ -17,5 +17,5 @@
         odometry_topic="odom"
         odom_frame="odom"
-        base_frame="base_footprint"
+        base_frame="base_link"
         max_wheel_torque="200"
         max_acceleration="1.0"
